File: RasPoE/RasPoE.kicad_pcb (KiCad board)
At the start: 2 copper layers, 85 x 56 mm, 46 parts, among them J1 RJSSE-5080, J2 RJSSE-5380, P1 CONN_02X20, P101 CONN_01X01, P102 CONN_01X01, P2 CONN_01X02, U1 AG9800

Commit message: Cosmetic touchups
Other:
- board text added: "Disconnect cable to RasPi before disconnecting powered PoE cable!"
- board text added: "RasPoE RasPi PoE shield for B+/2B v1.0"
- board text removed: "RasPoE RasPi PoE shield for B+/2B"

Commit message: Cleanup schematic
Parts:
- C10: value 10n -> 100n
- F1: value FUSE -> PTC 1A25; footprint Resistors_SMD:R_0805_HandSoldering -> Resistors_SMD:R_1812
- FB1, FB2, FB3, FB5, FB7, FB8: value FILTER -> WE 742792651
- P101, P102: value CONN_01X01 -> Wire pad
- P2: value CONN_01X02 -> Screw terminal 2.54mm
- TR1: value 749012011 -> WE_749012011
- U1: value AG9800 -> AG9805-MT
- moved FID2 1.69 mm to (36.8, 41.3)
- moved F1 1.34 mm to (42.0, 42.5)
- moved C6 0.54 mm to (52.0, 47.0)
Connections:
- B1 pad 2: /POE_A+ -> /POE_A-
- B1 pad 4: /POE_A- -> /POE_A+
- C4 pad 1: /POE_A- -> /POE_A+
- C5 pad 1: /POE_A+ -> /POE_A-
- D1 pad 1: /AG_IN_- -> /AG_IN_+
- D1 pad 2: /AG_IN_+ -> /AG_IN_-
- D2 pad 1: Net-(D2-Pad1) -> GND
- D2 pad 2: GND -> Net-(D2-Pad2)
- R5 pad 2: Net-(D2-Pad1) -> Net-(D2-Pad2)
- R8 pad 1: /AG_OUT+ -> /AG_OUT_+
- TR1 pad 2: /POE_A- -> /POE_A+
- TR1 pad 5: /POE_A+ -> /POE_A-
Routing:
- net /AG_OUT+: track 14.2 -> 0.00 mm, vias 2 -> 0
- net /POE_A-: track 47.1 -> 55.2 mm
- net /POE_A+: track 55.2 -> 47.1 mm
- net /AG_OUT_+: track 10.8 -> 14.2 mm, vias 0 -> 2
- net Net-(D2-Pad2): track 0.00 -> 2.43 mm
- net Net-(D2-Pad1): track 2.43 -> 0.00 mm
Other:
- board text added: "1A25"
- board text added: "RasPoE 1.0 PoE shield for B+/2B"
- board text removed: "1A1"
- board text removed: "Disconnect cable to RasPi before disconnecting powered PoE cable!"
- board text removed: "RasPoE RasPi PoE shield for B+/2B v1.0"
